File: PCB-design/MX43.kicad_pcb (KiCad board)
At the start: 2 copper layers, 238.8 x 86.4 mm, 116 parts, among them J1 Conn_01x12, J2 Conn_01x12, U1 CherryMX_LTST-A683CEGBW, U10 CherryMX_LTST-A683CEGBW, U11 CherryMX_LTST-A683CEGBW, U12 CherryMX_LTST-A683CEGBW, U13 CherryMX_LTST-A683CEGBW, U14 CherryMX_LTST-A683CEGBW, U15 CherryMX_LTST-A683CEGBW, U16 CherryMX_LTST-A683CEGBW, U17 CherryMX_LTST-A683CEGBW, U18 CherryMX_LTST-A683CEGBW, U19 CherryMX_LTST-A683CEGBW, U2 CherryMX_LTST-A683CEGBW, U20 CherryMX_LTST-A683CEGBW, U21 CherryMX_LTST-A683CEGBW, U22 CherryMX_LTST-A683CEGBW, U23 CherryMX_LTST-A683CEGBW, U24 CherryMX_LTST-A683CEGBW, U25 CherryMX_LTST-A683CEGBW, U26 CherryMX_LTST-A683CEGBW, U27 CherryMX_LTST-A683CEGBW, U28 CherryMX_LTST-A683CEGBW, U29 CherryMX_LTST-A683CEGBW, U3 CherryMX_LTST-A683CEGBW, U30 CherryMX_LTST-A683CEGBW, U31 CherryMX_LTST-A683CEGBW, U32 CherryMX_LTST-A683CEGBW, U33 CherryMX_LTST-A683CEGBW, U34 CherryMX_LTST-A683CEGBW, U35 CherryMX_LTST-A683CEGBW, U36 CherryMX_LTST-A683CEGBW, U37 CherryMX_LTST-A683CEGBW, U38 CherryMX_LTST-A683CEGBW, U39 CherryMX_LTST-A683CEGBW, U4 CherryMX_LTST-A683CEGBW, U40 CherryMX_LTST-A683CEGBW, U41 CherryMX_LTST-A683CEGBW, U42 CherryMX_LTST-A683CEGBW, U43 CherryMX_LTST-A683CEGBW, U5 CherryMX_LTST-A683CEGBW, U6 CherryMX_LTST-A683CEGBW, U7 CherryMX_LTST-A683CEGBW, U8 CherryMX_LTST-A683CEGBW, U9 CherryMX_LTST-A683CEGBW

Commit message: minor  updates
Parts:
- U24: footprint CherryMX_KailhSocket_StabWireTop_LTST-A683CEGBW-Rotated:CherryMX_2.00u_KailhSocket_StabWireTop_LTST-A683CEGBW-Rotated -> CherryMX_PCB_KailhSocket_StabWireBottom_LTST-A683CEGBW-Rotated:CherryMX_2.00u_PCB_KailhSocket_StabWireBottom_LTST-A683C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
- U38: footprint CherryMX_KailhSocket_StabWireTop_LTST-A683CEGBW-Rotated:CherryMX_2.75u_KailhSocket_StabWireTop_LTST-A683CEGBW-Rotated -> CherryMX_PCB_KailhSocket_StabWireBottom_LTST-A683CEGBW-Rotated:CherryMX_2.75u_PCB_KailhSocket_StabWireBottom_LTST-A683C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
- U39: footprint CherryMX_KailhSocket_StabWireTop_LTST-A683CEGBW-Rotated:CherryMX_2.25u_KailhSocket_StabWireTop_LTST-A683CEGBW-Rotated -> CherryMX_PCB_KailhSocket_StabWireBottom_LTST-A683CEGBW-Rotated:CherryMX_2.25u_PCB_KailhSocket_StabWireBottom_LTST-A683C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
Routing:
- net ROW2: track 230.1 -> 232.2 mm
- net VCC: track 1092.8 -> 1094.8 mm
- net RGBDataR4: track 248.8 -> 250.6 mm
- net ROW1: track 262.1 -> 263.4 mm
- net GND: track 96.3 -> 96.1 mm, vias 63 -> 62
Other:
- board text added: "License: CERN-OHL-W https://github.com/jpconstantineau/OffsetMX43 2021-09-28"
- board text removed: "License: CERN-OHL-W https://github.com/jpconstantineau/OffsetMX43 2021-09-02"
