File: PCB-design/MX43.sch (KiCad schematic (older format))
At the start: 116 parts, among them J1 Conn_01x12, J2 Conn_01x12, U1 CherryMX_LTST-A683CEGBW, U10 CherryMX_LTST-A683CEGBW, U11 CherryMX_LTST-A683CEGBW, U12 CherryMX_LTST-A683CEGBW, U13 CherryMX_LTST-A683CEGBW, U14 CherryMX_LTST-A683CEGBW, U15 CherryMX_LTST-A683CEGBW, U16 CherryMX_LTST-A683CEGBW, U17 CherryMX_LTST-A683CEGBW, U18 CherryMX_LTST-A683CEGBW, U19 CherryMX_LTST-A683CEGBW, U2 CherryMX_LTST-A683CEGBW, U20 CherryMX_LTST-A683CEGBW, U21 CherryMX_LTST-A683CEGBW, U22 CherryMX_LTST-A683CEGBW, U23 CherryMX_LTST-A683CEGBW, U24 CherryMX_LTST-A683CEGBW, U25 CherryMX_LTST-A683CEGBW, U26 CherryMX_LTST-A683CEGBW, U27 CherryMX_LTST-A683CEGBW, U28 CherryMX_LTST-A683CEGBW, U29 CherryMX_LTST-A683CEGBW, U3 CherryMX_LTST-A683CEGBW, U30 CherryMX_LTST-A683CEGBW, U31 CherryMX_LTST-A683CEGBW, U32 CherryMX_LTST-A683CEGBW, U33 CherryMX_LTST-A683CEGBW, U34 CherryMX_LTST-A683CEGBW, U35 CherryMX_LTST-A683CEGBW, U36 CherryMX_LTST-A683CEGBW, U37 CherryMX_LTST-A683CEGBW, U38 CherryMX_LTST-A683CEGBW, U39 CherryMX_LTST-A683CEGBW, U4 CherryMX_LTST-A683CEGBW, U40 CherryMX_LTST-A683CEGBW, U41 CherryMX_LTST-A683CEGBW, U42 CherryMX_LTST-A683CEGBW, U43 CherryMX_LTST-A683CEGBW, U5 CherryMX_LTST-A683CEGBW, U6 CherryMX_LTST-A683CEGBW, U7 CherryMX_LTST-A683CEGBW, U8 CherryMX_LTST-A683CEGBW, U9 CherryMX_LTST-A683CEGBW

Commit message: minor  updates
Parts:
- U24: footprint CherryMX_KailhSocket_StabWireTop_LTST-A683CEGBW-Rotated:CherryMX_2.00u_KailhSocket_StabWireTop_LTST-A683CEGBW-Rotated -> CherryMX_PCB_KailhSocket_StabWireBottom_LTST-A683CEGBW-Rotated:CherryMX_2.00u_PCB_KailhSocket_StabWireBottom_LTST-A683C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
- U38: footprint CherryMX_KailhSocket_StabWireTop_LTST-A683CEGBW-Rotated:CherryMX_2.75u_KailhSocket_StabWireTop_LTST-A683CEGBW-Rotated -> CherryMX_PCB_KailhSocket_StabWireBottom_LTST-A683CEGBW-Rotated:CherryMX_2.75u_PCB_KailhSocket_StabWireBottom_LTST-A683C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
- U39: footprint CherryMX_KailhSocket_StabWireTop_LTST-A683CEGBW-Rotated:CherryMX_2.25u_KailhSocket_StabWireTop_LTST-A683CEGBW-Rotated -> CherryMX_PCB_KailhSocket_StabWireBottom_LTST-A683CEGBW-Rotated:CherryMX_2.25u_PCB_KailhSocket_StabWireBottom_LTST-A683C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
Changed lines of the file:
@@
 F 0 "U38" H 6350 4535 50  0000 C CNN
 F 1 "CherryMX_LTST-A683CEGBW" H 6350 4444 50  0000 C CNN
-F 2 "CherryMX_KailhSocket_StabWireTop_LTST-A683CEGBW-Rotated:CherryMX_2.75u_KailhSocket_StabWireTop_LTST-A683CEGBW-Rotated" H 6350 4050 50  0001 C CNN
+F 2 "CherryMX_PCB_KailhSocket_StabWireBottom_LTST-A683CEGBW-Rotated:CherryMX_2.75u_PCB_KailhSocket_StabWireBottom_LTST-A683CEGBW-Rotated" H 6350 4050 50  0001 C CNN
 F 3 "" H 6350 4050 50  0001 C CNN
 	1    6350 4150
@@
 F 0 "U24" H 1850 3635 50  0000 C CNN
 F 1 "CherryMX_LTST-A683CEGBW" H 1850 3544 50  0000 C CNN
-F 2 "CherryMX_KailhSocket_StabWireTop_LTST-A683CEGBW-Rotated:CherryMX_2.00u_KailhSocket_StabWireTop_LTST-A683CEGBW-Rotated" H 1850 3150 50  0001 C CNN
+F 2 "CherryMX_PCB_KailhSocket_StabWireBottom_LTST-A683CEGBW-Rotated:CherryMX_2.00u_PCB_KailhSocket_StabWireBottom_LTST-A683CEGBW-Rotated" H 1850 3150 50  0001 C CNN
 F 3 "" H 1850 3150 50  0001 C CNN
 	1    1850 3250
@@
 F 0 "U39" H 7800 4535 50  0000 C CNN
 F 1 "CherryMX_LTST-A683CEGBW" H 7800 4444 50  0000 C CNN
-F 2 "CherryMX_KailhSocket_StabWireTop_LTST-A683CEGBW-Rotated:CherryMX_2.25u_KailhSocket_StabWireTop_LTST-A683CEGBW-Rotated" H 7800 4050 50  0001 C CNN
+F 2 "CherryMX_PCB_KailhSocket_StabWireBottom_LTST-A683CEGBW-Rotated:CherryMX_2.25u_PCB_KailhSocket_StabWireBottom_LTST-A683CEGBW-Rotated" H 7800 4050 50  0001 C CNN
 F 3 "" H 7800 4050 50  0001 C CNN
 	1    7800 4150
